File: ModuleV400/v4.kicad_pcb (KiCad board)
At the start: 2 copper layers, 30 x 50 mm, 42 parts, among them J2 AVR-ISP-6, Q1 IRLML6244TRPBF, U1 HMHA2801, U4 ATtiny841-SSU

Commit message: Kicad cleanup, new power dissipation layout (#114)
* Update module v440 to Kicad 6.
* V4.4 PCB design update

Changes:

* reconnect a couple of misaligned vias
* move non-power routes (PTC, bypass switch transistor) off the heat dissipation area
* add a lot of vias and copper to resistor array, for improved heat dissipation
* rearranged resistor array for more connections == larger copper area
* moved the slit up a bit for more room in heat dissipation area
* added "not in schematic" tags to the mount holes

Component values and placement have NOT changed.
(Exception: parts of the resistor array have switched places. That's obviously harmless.)

* Updated for Kicad 6

The schematic has NOT been realigned.

* added "not in schematic" tag to the mounting holes
* Imported V400 to Kicad 6.

The schematic has NOT been realigned.

* added not-in-schematic tags to the mounting holes.
* Minor cleanup
* Switch to kicad 6.0
* Updated date and version#
Other:
- net class Default removed
- net class Power removed
